Commit message: いったん自環境をコミット パスとかおかしくなってるかも？

File: 2018/catkin_ws/src/my_robo/my_robo_description/my_robo.urdf (robot description, URDF)
Before this commit: robot my_robo, 5 links, 4 joints
Links:
- added link hokuyo_link, mass 1e-5; collision box size=0.1 0.1 0.1; visual mesh filename=package://rrbot_description/meshes/hokuyo.dae
Joints:
- added joint hokuyo_joint: type fixed, parent base_link, child hokuyo_link, origin xyz=0.2 0 0.07 rpy=0 0 0, axis 0 1 0
